File: SolarCore.kicad_sch (KiCad schematic)
At the start: 10 parts, among them U1 LMR33630ARNXR

Commit message: Schematic update V1
Parts:
- added C6, C7, C8: 22u, symbol Device:C
- C1, C2: value C -> 4.7u
- C4: value C -> 22u
Connections:
- net GND: now also C6.1, C7.1, C8.1
- net V_OUT: now also C6.2, C7.2, C8.2

Commit message: Schematic update V2
Parts:
- added C10, C9: 100n, symbol Device:C
Connections:
- net GND: now also C10.2, C9.2
- net V_IN: now also C10.1, C9.1
Other:
- moved on the sheet: C1, C2, C3, C4, C5, C6, C7, C8, L1, R1, R2, R3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
