File: KiCAD/SolarCore.kicad_sch (KiCad schematic)
At the start: 29 parts, among them J1 Conn_01x02_MountingPin, J2 Conn_01x02_MountingPin, SW1 SW_SPST, U1 LMR33630ARNXR, U2 NUCLEO-L432KC

Commit message: Final schematic V4
Parts:
- R4: value 200k -> 100k
- R7: value 200k -> 75k
- R8: value 100k -> 27k
Changed lines of the file:
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@@
 			)
 		)
-		(property "Value" "200k"
+		(property "Value" "100k"
 			(at 308.61 175.2599 0)
 			(effects
@@
 			)
 		)
-		(property "Value" "100k"
+		(property "Value" "27k"
 			(at 114.3 187.9599 0)
 			(effects
@@
 			)
 		)
-		(property "Value" "200k"
+		(property "Value" "75k"
 			(at 114.3 175.2599 0)
 			(effects

Commit message: Final schematic V5
Parts:
- added NT1: NetTie_2, NetTie:NetTie-2_SMD_Pad0.5mm, symbol Device:NetTie_2
Connections:
- net GND: now also NT1.2; no longer C1.2, C10.2, C2.2, C4.1, C6.1, C7.1, C8.1, C9.2, D1.2 (A), J1.2 (Pin_2), J2.2 (Pin_2), R2.2, U1.1 (PGND)
- new net PGND: C1.2, C10.2, C2.2, C4.1, C6.1, C7.1, C8.1, C9.2, D1.2 (A), J1.2 (Pin_2), J2.2 (Pin_2), NT1.1, R2.2, U1.1 (PGND)
