File: KiCAD/SolarCore.kicad_pcb (KiCad board)
At the start: 2 copper layers, 30 parts, among them J1 Conn_01x02_MountingPin, J2 Conn_01x02_MountingPin, SW1 SW_SPST, U1 LMR33630ARNXR, U2 NUCLEO-L432KC

Commit message: PCB V2
Parts:
- moved C4 47.3 mm to (178.9, 105.6)
- moved F1 46.9 mm to (127.1, 75.1)
- moved U1 45.3 mm to (174.2, 75.3), turned to 180 degrees
- moved C6 43.0 mm to (178.9, 99.1)
- moved NT1 42.3 mm to (171.4, 80.4)
- moved C7 42.0 mm to (178.9, 92.6)
- moved J2 41.9 mm to (177.1, 113.3)
- moved L1 41.7 mm to (175.6, 80.4), turned to -90 degrees
- moved C8 36.9 mm to (178.8, 86.1)
- moved D1 34.4 mm to (144.1, 78.6), turned to -90 degrees
- moved J1 30.6 mm to (124.1, 83.6), turned to -90 degrees
- moved SW1 30.5 mm to (133.9, 75.4)
- moved R1 30.1 mm to (180.9, 80.6), turned to 90 degrees
- moved R2 27.8 mm to (181.9, 77.6)
- moved C3 26.8 mm to (177.1, 75.4), turned to -90 degrees
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Connections:
- C4 pad 1: PGND -> V_OUT_MEAS
- C4 pad 2: V_OUT_MEAS -> PGND
- C6 pad 1: PGND -> V_OUT_MEAS
- C6 pad 2: V_OUT_MEAS -> PGND
- C7 pad 1: PGND -> V_OUT_MEAS
- C7 pad 2: V_OUT_MEAS -> PGND
- C8 pad 1: PGND -> V_OUT_MEAS
- C8 pad 2: V_OUT_MEAS -> PGND
Other:
- copper layers 2 -> 4

Commit message: PCB V3
Parts:
- moved C11 4.91 mm to (169.2, 83.5), turned to 0 degrees
- moved J1 1.15 mm to (123.0, 83.5)
- moved R1 1.07 mm to (181.9, 80.2), turned to 180 degrees
- moved U2 0.57 mm to (146.1, 100.6)
- moved C3 0.40 mm to (177.5, 75.4), turned to 0 degrees
Routing:
- net V_OUT_MEAS: track 0.34 -> 32.3 mm
- net V_IN_MEAS: track 0.00 -> 30.9 mm
- net Net-(J1-Pin_1): track 0.00 -> 6.29 mm
- net Net-(SW1-A): track 0.00 -> 3.91 mm

Commit message: PCB V4
Parts:
- added REF**: MountingHole_2.7mm_M2.5, MountingHole:MountingHole_2.7mm_M2.5, F.Cu at (123.0, 124.2)
- added REF**: MountingHole_2.7mm_M2.5, MountingHole:MountingHole_2.7mm_M2.5, F.Cu at (193.0, 69.2)
- added REF**: MountingHole_2.7mm_M2.5, MountingHole:MountingHole_2.7mm_M2.5, F.Cu at (192.8, 124.2)
- added REF**: MountingHole_2.7mm_M2.5, MountingHole:MountingHole_2.7mm_M2.5, F.Cu at (123.2, 69.2)
- moved C1 7.59 mm to (151.2, 84.9)
- moved C10 7.59 mm to (169.7, 84.9)
- moved C12 7.59 mm to (151.9, 75.4)
- moved C2 7.59 mm to (157.2, 84.9)
- moved C3 7.59 mm to (178.6, 82.9)
- moved C4 7.59 mm to (179.9, 113.1)
- moved C5 7.59 mm to (175.5, 76.4)
- moved C6 7.59 mm to (179.9, 106.6)
- moved C7 7.59 mm to (179.9, 100.1)
- moved C8 7.59 mm to (179.9, 93.6)
- moved C9 7.59 mm to (163.2, 84.8)
- moved D1 7.59 mm to (145.2, 86.1)
- moved J1 7.59 mm to (124.1, 91.0)
- moved J2 7.59 mm to (178.2, 120.8)
- moved L1 7.59 mm to (176.7, 87.9)
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Routing:
- net PA1: track 0.00 -> 24.6 mm, vias 0 -> 2
- net Net-(U1-FB): track 0.00 -> 12.5 mm, vias 0 -> 2
- net PA0: track 0.00 -> 11.8 mm
- net V_OUT_MEAS: track 32.3 -> 43.7 mm
- net V_IN_MEAS: track 30.9 -> 37.8 mm
- net Net-(R4-Pad2): track 0.00 -> 5.85 mm
- net Net-(U1-VCC): track 0.00 -> 5.64 mm
- net Net-(R7-Pad2): track 0.00 -> 5.34 mm
- net Net-(U1-SW): track 0.00 -> 4.49 mm
- net PG: track 0.00 -> 3.35 mm
- net Net-(C12-Pad1): track 0.00 -> 3.13 mm
- net Net-(C11-Pad1): track 0.00 -> 2.66 mm
- net Net-(U1-BST): track 0.00 -> 1.84 mm
